File: PCB/heartbeat/heartbeat.kicad_sch (KiCad schematic)
At the start: 17 parts, among them J1 USB_C_Receptacle, J2 AudioJack3, U1 ESP32-WROOM-32, U2 AMS1117-3.3, U3 CH330N, U4 LM358_DFN

Commit message: addec missing componments
Parts:
- added D1: Inolux_IN-P55TATRGB, LED_SMD:LED_Inolux_IN-P55TATRGB_PLCC6_5.0x5.5mm_P1.8mm, symbol LED:Inolux_IN-P55TATRGB
- added J3: Conn_01x02, Connector_JST:JST_PH_S2B-PH-K_1x02_P2.00mm_Horizontal, symbol Connector_Generic:Conn_01x02
- added U5: LGS5500EP, Package_SO:SOIC-8-1EP_3.9x4.9mm_P1.27mm_EP2.41x3.3mm, symbol Battery_Management:LGS5500EP
Connections:
- net 5V: now also U5.2 (VIN)
